File: Table_Controller.kicad_sch (KiCad schematic)
At the start: 169 parts, among them J10 1050171001 Micro Type B, J11 HX JN1.27-2x5 WZ H4.9, J12 Conn_01x04_Pin, J13 Conn_01x14_Pin, J14 2.54 mm header, J15 2.54 mm header, U10 STM32G431K8Tx, U11 LMR380x0, U12 VNH7070, Y10 20 MHz

Commit message: sch drafted, missing power input connector
Parts:
- J11: footprint Personal:JN1.27-2x5 WZ H4.9 -> Personal:HX JN1.27-2x5P ZZ H4.9
Changed lines of the file:
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@@
 	)
 	(junction
-		(at 101.6 151.13)
+		(at 77.47 39.37)
 		(diameter 0)
 		(color 0 0 0 0)
 	)
 	(junction
-		(at 77.47 39.37)
+		(at 166.37 151.13)
 		(diameter 0)
 		(color 0 0 0 0)
@@
 	)
 	(junction
+		(at 50.8 161.29)
+		(diameter 0)
+		(color 0 0 0 0)
+	)
+	(junction
 		(at 264.16 54.61)
 		(diameter 0)
@@
 	)
 	(junction
-		(at 166.37 151.13)
+		(at 88.9 161.29)
 		(diameter 0)
 		(color 0 0 0 0)
@@
 	)
 	(junction
+		(at 119.38 151.13)
+		(diameter 0)
+		(color 0 0 0 0)
+	)
+	(junction
 		(at 251.46 76.2)
 		(diameter 0)
@@
 	)
 	(junction
-		(at 119.38 151.13)
+		(at 125.73 161.29)
 		(diameter 0)
 		(color 0 0 0 0)
 	)
 	(junction
-		(at 125.73 161.29)
+		(at 101.6 151.13)
 		(diameter 0)
 		(color 0 0 0 0)
@@
 	)
 	(junction
-		(at 50.8 161.29)
-		(diameter 0)
-		(color 0 0 0 0)
-	)
-	(junction
 		(at 191.77 30.48)
 		(diameter 0)
@@
 	)
 	(junction
-		(at 88.9 161.29)
-		(diameter 0)
-		(color 0 0 0 0)
-	)
-	(junction
 		(at 240.03 104.14)
 		(diameter 0)
@@
 	(wire
 		(pts
+			(xy 166.37 151.13) (xy 167.64 151.13)
+		)
+		(stroke
+			(width 0)
+			(type default)
+		)
+	)
+	(wire
+		(pts
 			(xy 29.21 90.17) (xy 29.21 100.33)
 		)
@@
 	(wire
 		(pts
+			(xy 88.9 161.29) (xy 115.57 161.29)
+		)
+		(stroke
+			(width 0)
+			(type default)
+		)
+	)
+	(wire
+		(pts
 			(xy 20.32 133.35) (xy 31.75 133.35)
 		)
@@
 	(wire
 		(pts
-			(xy 105.41 151.13) (xy 101.6 151.13)
-		)
-		(stroke
-			(width 0)
-			(type default)
-		)
-	)
-	(wire
-		(pts
 			(xy 77.47 39.37) (xy 77.47 57.15)
 		)
@@
 	(wire
 		(pts
+			(xy 119.38 151.13) (xy 125.73 151.13)
+		)
+		(stroke
+			(width 0)
+			(type default)
+		)
+	)
+	(wire
+		(pts
 			(xy 48.26 31.75) (xy 64.77 31.75)
 		)
@@
 	(wire
 		(pts
-			(xy 101.6 151.13) (xy 88.9 151.13)
+			(xy 88.9 151.13) (xy 101.6 151.13)
 		)
 		(stroke
@@
 	(wire
 		(pts
+			(xy 101.6 151.13) (xy 105.41 151.13)
+		)
+		(stroke
+			(width 0)
+			(type default)
+		)
+	)
+	(wire
+		(pts
 			(xy 19.05 132.08) (xy 19.05 133.35)
 		)
@@
 	(wire
 		(pts
-			(xy 119.38 151.13) (xy 125.73 151.13)
-		)
-		(stroke
-			(width 0)
-			(type default)
-		)
-	)
-	(wire
-		(pts
 			(xy 43.18 133.35) (xy 54.61 133.35)
 		)
@@
 	(wire
 		(pts
-			(xy 88.9 161.29) (xy 115.57 161.29)
-		)
-		(stroke
-			(width 0)
-			(type default)
-		)
-	)
-	(wire
-		(pts
 			(xy 259.08 101.6) (xy 259.08 105.41)
 		)
@@
 	(wire
 		(pts
-			(xy 167.64 151.13) (xy 166.37 151.13)
-		)
-		(stroke
-			(width 0)
-			(type default)
-		)
-	)
-	(wire
-		(pts
 			(xy 74.93 170.18) (xy 73.66 170.18)
 		)
@@
 			)
 		)
-		(property "Footprint" "Personal:JN1.27-2x5 WZ H4.9"
+		(property "Footprint" "Personal:HX JN1.27-2x5P ZZ H4.9"
 			(at 212.09 139.7 0)
 			(hide yes)
