File: Table_Controller.kicad_pcb (KiCad board)
At the start: 4 copper layers, 100.6 x 50 mm, 102 parts, among them J1 Dell DC jack, J11 HX JN1.27-2x5 WZ H4.9, J12 JST B4B XH A, J13 Conn_01x14_Pin, J14 JST B6B XH A, J15 2.54 mm header, J2 USB_C_Receptacle_USB2.0_16P, J3 DC barrel assy, U1 USBLC6-2SC6, U10 STM32G431K8Tx, U11 LMR380x0, U12 VNH7070, Y10 20 MHz

Commit message: routing 50%
Parts:
- removed H10, H11, H12, H13, H14, H15: MountingHole, MountingHole:MountingHole_3.2mm_M3
- removed JP45: 0R, Personal:Jumper_0603
- added JP28: 0R, Resistor_THT:R_Axial_DIN0204_L3.6mm_D1.6mm_P7.62mm_Horizontal, F.Cu at (40.6, 47.2)
- moved JP27 98.3 mm to (38.4, 49.0)
- moved TP29 98.2 mm to (76.7, 27.9)
- moved C18 98.1 mm to (32.2, 20.2)
- moved C26 98.1 mm to (36.9, 28.6)
- moved TP14 98.1 mm to (28.9, 19.9)
- moved C14 98.1 mm to (38.4, 20.0)
- moved C16 98.1 mm to (35.7, 20.0)
- moved C20 98.1 mm to (30.8, 32.1)
- moved C22 98.1 mm to (30.4, 36.0)
- moved C28 98.1 mm to (37.2, 24.5)
- moved L10 98.1 mm to (35.9, 34.0)
- moved R12 98.1 mm to (27.4, 22.6)
- moved R13 98.1 mm to (28.4, 36.0)
- moved R14 98.1 mm to (27.6, 27.4)
- moved TP13 98.1 mm to (29.0, 30.4)
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Routing:
- net /GND: track 14.4 -> 42.3 mm, vias 32 -> 57
- net /S19V5: track 65.2 -> 38.8 mm
- net /SEL0': track 23.7 -> 2.27 mm, vias 2 -> 0
- net /S3V3: track 318.5 -> 339.8 mm
- net /OUTa: track 18.6 -> 0.00 mm
- net /SEL0: track 19.3 -> 37.7 mm
- net /SWO': track 10.3 -> 0.00 mm
- net /OUTb: track 9.58 -> 0.00 mm
- net /OUTb': track 8.62 -> 0.07 mm
- net /CS': track 10.9 -> 15.2 mm
- net Net-(J13-Pin_14): track 0.00 -> 4.19 mm
- net Net-(J13-Pin_13): track 0.00 -> 3.88 mm
- net Net-(J13-Pin_7): track 0.00 -> 3.69 mm
- net Net-(J13-Pin_10): track 0.00 -> 3.58 mm
- net Net-(J13-Pin_11): track 0.00 -> 3.58 mm
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- added copper zone on F.Cu, net /GND
- added copper zone on F.Cu, net /OUTa
- added copper zone on F.Cu, net /OUTb
- added copper zone on F.Cu, net /OUTb'
Other:
- board size 100.6 x 50 mm -> 103.1 x 50 mm

Commit message: routing 75%
Parts:
- moved TP24 10.6 mm to (41.1, 18.0)
- moved TP25 9.09 mm to (58.7, 17.5)
- moved JP38 5.24 mm to (42.2, 23.4)
- moved J11 1.59 mm to (52.5, 23.8)
- moved R24 1.50 mm to (58.9, 23.6)
- moved JP47 1.39 mm to (62.7, 27.7)
- moved J2 1.23 mm to (62.7, 21.6)
- moved R23 1.19 mm to (66.5, 19.6)
- moved U1 0.72 mm to (66.3, 29.0)
Routing:
- net Net-(J2-VBUS-PadA4): track 5.79 -> 19.1 mm
- net /SWO': track 0.00 -> 10.3 mm
- net /S3V3: track 339.8 -> 334.6 mm
- net /GND: track 42.3 -> 47.3 mm
- net /D-: track 8.25 -> 12.7 mm
- net /3V3_REG: track 28.9 -> 25.1 mm
- net /D+: track 17.5 -> 14.8 mm
- net /D-': track 0.00 -> 2.15 mm
- net /D+': track 3.61 -> 1.75 mm
- net /SWDCLK: track 24.1 -> 22.4 mm
- net /SWDIO: track 28.2 -> 26.6 mm
- net /USB_DM: track 5.19 -> 5.89 mm
