File: Table_Controller_DCDC_rotated.kicad_pcb (KiCad board)
At the start: 4 copper layers, 103.1 x 50 mm, 96 parts, among them J1 Dell DC jack, J11 HX JN1.27-2x5 WZ H4.9, J12 JST B4B XH A, J13 Conn_01x14_Pin, J14 JST B6B XH A, J15 2.54 mm header, J2 USB_C_Receptacle_USB2.0_16P, J3 DC barrel assy, U1 USBLC6-2SC6, U10 STM32G431K8Tx, U11 LMR380x0, U12 VNH7070, Y10 20 MHz

Commit message: layout option 1 done
Parts:
- moved R13 19.3 mm to (39.6, 21.8), turned to -90 degrees
- moved C22 16.9 mm to (37.8, 21.8), turned to -90 degrees
- moved TP14 16.9 mm to (38.1, 34.8), turned to 90 degrees
- moved TP24 15.9 mm to (26.7, 33.5), turned to 90 degrees
- moved R12 15.9 mm to (39.6, 32.0), turned to 90 degrees
- moved TP16 15.8 mm to (39.6, 24.9), turned to 90 degrees
- moved C24 15.6 mm to (24.9, 26.9), turned to 180 degrees
- moved TP17 15.5 mm to (24.9, 29.7), turned to 90 degrees
- moved TP15 15.2 mm to (35.8, 21.6), turned to 90 degrees
- moved R14 14.2 mm to (39.6, 27.9), turned to -90 degrees
- moved L10 14.2 mm to (30.7, 21.6), turned to 180 degrees
- moved C14 14.0 mm to (29.2, 34.6), turned to 90 degrees
- moved C18 13.7 mm to (35.1, 34.8), turned to 180 degrees
- moved JP38 12.4 mm to (26.7, 30.5), turned to -90 degrees
- moved C16 12.3 mm to (31.8, 34.5), turned to 90 degrees
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Routing:
- net /S19V5: track 54.2 -> 20.0 mm
- net /S3V3: track 362.6 -> 367.4 mm
- net /GND: track 56.8 -> 58.2 mm
