File: Table_Controller_Vin_edge.kicad_pcb (KiCad board)
At the start: 4 copper layers, 103.1 x 50 mm, 96 parts, among them J1 Dell DC jack, J11 HX JN1.27-2x5 WZ H4.9, J12 JST B4B XH A, J13 Conn_01x14_Pin, J14 JST B6B XH A, J15 2.54 mm header, J2 USB_C_Receptacle_USB2.0_16P, J3 DC barrel assy, U1 USBLC6-2SC6, U10 STM32G431K8Tx, U11 LMR380x0, U12 VNH7070, Y10 20 MHz

Commit message: top silk done
Parts:
- moved R13 19.3 mm to (25.5, 35.0), turned to 90 degrees
- moved C22 16.9 mm to (27.2, 35.0), turned to 90 degrees
- moved TP14 16.9 mm to (27.0, 22.1), turned to -90 degrees
- moved TP24 15.9 mm to (40.2, 25.1), turned to -90 degrees
- moved R12 15.9 mm to (25.5, 24.9), turned to -90 degrees
- moved TP16 15.8 mm to (25.5, 32.0), turned to -90 degrees
- moved C24 15.6 mm to (40.2, 29.9), turned to 0 degrees
- moved TP17 15.5 mm to (40.2, 27.1), turned to -90 degrees
- moved TP15 15.2 mm to (29.3, 35.3), turned to -90 degrees
- moved R14 14.2 mm to (25.5, 28.9), turned to 90 degrees
- moved L10 14.2 mm to (34.3, 35.3), turned to 0 degrees
- moved C14 14.0 mm to (35.9, 22.3), turned to -90 degrees
- moved C18 13.7 mm to (30.0, 22.1), turned to 0 degrees
- moved JP38 12.4 mm to (38.4, 26.4), turned to 90 degrees
- moved C16 12.3 mm to (33.3, 22.3), turned to -90 degrees
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Routing:
- net /S19V5: track 20.0 -> 54.2 mm
- net /S3V3: track 367.4 -> 362.6 mm
- net /GND: track 58.2 -> 56.8 mm
