File: _restore_backup_2026-09-18T15-40-45-056/Table_Controller.kicad_sch (KiCad schematic)
At the start: 173 parts, among them J10 1050171001 Micro Type B, J11 HX JN1.27-2x5 WZ H4.9, J12 Conn_01x04_Pin, J13 Conn_01x14_Pin, J14 2.54 mm header, J15 2.54 mm header, U10 STM32G431K8Tx, U11 LMR380x0, U12 VNH7070, Y10 20 MHz

Commit message: Placement proposal 90%
Parts:
- removed JP19, JP31: 0R, Resistor_THT:R_Axial_DIN0204_L3.6mm_D1.6mm_P5.08mm_Horizontal, symbol Device:R
- removed JP32: 0R, Resistor_THT:R_Axial_DIN0204_L3.6mm_D1.6mm_P7.62mm_Horizontal, symbol Device:R
- removed JP34, JP35, JP36, JP37, JP38, JP39, JP40, JP41, JP42, JP43, JP44, JP45, JP46: 0R, Personal:Jumper_0603, symbol Device:R
- added JP10, JP11, JP12, JP13, JP14, JP20, JP21, JP22, JP23, JP28, JP30: 0R, Resistor_SMD:R_0603_1608Metric_Pad0.98x0.95mm_HandSolder, symbol Device:R
- added JP18: 0R, Resistor_THT:R_Axial_DIN0204_L3.6mm_D1.6mm_P5.08mm_Horizontal, symbol Device:R
- JP25, JP26, JP27: footprint Resistor_THT:R_Axial_DIN0204_L3.6mm_D1.6mm_P7.62mm_Horizontal -> Resistor_SMD:R_0603_1608Metric_Pad0.98x0.95mm_HandSolder; Manufacturer Generic -> Yageo; Manufacturer Part Number Hand cut wire -> RC0603JR-130RP
Connections:
- net DISP_CS: now also JP25.1
- net DISP_MISO: now also JP13.1
- net DISP_MOSI: now also JP14.1, JP18.1
- net DISP_RST: now also JP20.1
- net INa: now also JP26.1; no longer TP19.1
- net INb: now also JP27.1; no longer JP26.2, TP20.1
- net OUTa: now also U12.15 (OUTa), U12.2 (OUTa); no longer JP27.1
- net PWM: now also P18.1, U10.27 (PB4), JP28.1; no longer P38.1, TP21.1, U10.25 (PA15)
- net S19V5: now also C25.1, C27.1, U12.12 (VCC), U12.4 (VCC), U12.5 (VCC)
- net S3V3: now also JP12.1, JP21.2, JP22.1
- net S3V3_A: now also JP12.2
- net SEL0: now also P38.1, U10.25 (PA15), JP30.1; no longer P18.1, U10.27 (PB4)
- net SWO: now also J11.3 (Pin_3)
- net TCH_IRQ: now also JP23.1
- net USB_DM: now also JP11.2
- net USB_DP: now also JP10.2
- net at J13.4 (Pin_4): now also JP20.2
- net at J13.6 (Pin_6): now also JP18.2
- net at TP22.1, U12.14 (SEL0): now also JP30.2
- net at R15.2, R16.1: now also TP23.1, U12.13 (CS); no longer JP25.1
- net at J10.2 (D-): now also JP11.1
- net at J10.3 (D+): now also JP10.1
- net at C22.1, C24.1, C26.1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: now also JP21.1
- net at J14.4 (Pin_4): now also JP22.2
- net at U12.3 (INa): now also JP26.2, TP19.1
- net at J13.3 (Pin_3): now also JP25.2
- net at J13.12 (Pin_12): now also JP14.2
- net at J13.13 (Pin_13): now also JP13.2
- net at J13.14 (Pin_14): now also JP23.2
- net at U12.11 (PWM): now also TP21.1, JP28.2
- net at U12.6 (INb): now also JP27.2, TP20.1; no longer JP26.1
- net XIN: no longer names the net of C10.1, U10.2 (PF0), Y10.1
- net XOUT: no longer names the net of C13.1, U10.3 (PF1), Y10.3
Other:
- moved on the sheet: C25, C27, J11, TP19, TP20, TP21
